Commit message: fix inertial and collision

File: dream_walker_description/robots/dream_walker.urdf.xacro (robot description, xacro)
@@ -11,24 +11,28 @@
   <xacro:zero_leg prefix="A0" parent="base">
     <origin xyz="${joint_x0} -${joint_y0} ${joint_z0}" rpy="0 0 0"/>
-    <origin xyz="-${joint_x0} ${joint_y0} -${joint_z0}"/>
-    <origin xyz="${x0} -${y0} ${z0}"/>
-    <inertia ixx="${ixx0}" ixy="${ixy0}" ixz="${ixz0}" iyy="${iyy0}" iyz="${iyz0}" izz="${izz0}"/>
+    <origin xyz="-${visual_x0} ${visual_y0} -${visual_z0}"/>
+    <origin xyz="-${visual_x0} ${visual_y0} -${visual_z0}"/>
+    <origin xyz="-${x0} ${y0} ${z0}"/>
+    <inertia ixx="${ixx0}" ixy="-${ixy0}" ixz="${ixz0}" iyy="${iyy0}" iyz="${iyz0}" izz="${izz0}"/>
   </xacro:zero_leg>
   <xacro:zero_leg prefix="B0" parent="base">
     <origin xyz="${joint_x0} ${joint_y0} ${joint_z0}" rpy="0 0 0"/>
-    <origin xyz="-${joint_x0} -${joint_y0} -${joint_z0}"/>
-    <origin xyz="${x0} ${y0} ${z0}"/>
+    <origin xyz="-${visual_x0} -${visual_y0} -${visual_z0}"/>
+    <origin xyz="-${visual_x0} -${visual_y0} -${visual_z0}"/>
+    <origin xyz="-${x0} -${y0} ${z0}"/>
     <inertia ixx="${ixx0}" ixy="${ixy0}" ixz="${ixz0}" iyy="${iyy0}" iyz="${iyz0}" izz="${izz0}"/>
   </xacro:zero_leg>
   <xacro:zero_leg prefix="C0" parent="base">
     <origin xyz="-${joint_x0} -${joint_y0} ${joint_z0}" rpy="0 0 0"/>
-    <origin xyz="${joint_x0} ${joint_y0} -${joint_z0}"/>
-    <origin xyz="-${x0} -${y0} ${z0}"/>
+    <origin xyz="${visual_x0} ${visual_y0} -${visual_z0}"/>
+    <origin xyz="${visual_x0} ${visual_y0} -${visual_z0}"/>
+    <origin xyz="${x0} ${y0} ${z0}"/>
     <inertia ixx="${ixx0}" ixy="-${ixy0}" ixz="${ixz0}" iyy="${iyy0}" iyz="${iyz0}" izz="${izz0}"/>
   </xacro:zero_leg>
   <xacro:zero_leg prefix="D0" parent="base">
     <origin xyz="-${joint_x0} ${joint_y0} ${joint_z0}" rpy="0 0 0"/>
-    <origin xyz="${joint_x0} -${joint_y0} -${joint_z0}"/>
-    <origin xyz="-${x0} ${y0} ${z0}"/>
+    <origin xyz="${visual_x0} -${visual_y0} -${visual_z0}"/>
+    <origin xyz="${visual_x0} -${visual_y0} -${visual_z0}"/>
+    <origin xyz="${x0} -${y0} ${z0}"/>
     <inertia ixx="${ixx0}" ixy="-${ixy0}" ixz="${ixz0}" iyy="${iyy0}" iyz="${iyz0}" izz="${izz0}"/>
   </xacro:zero_leg>
@@ -36,5 +40,6 @@
     <origin xyz="${joint_x1} -${joint_y1} ${joint_z1}" rpy="0 0 0"/>
     <origin xyz="-${visual_x1} ${visual_y1} -${visual_z1}"/>
-    <origin xyz="${x1} -${y1} ${z1}"/>
+    <origin xyz="-${visual_x1} ${visual_y1} -${visual_z1}"/>
+    <origin xyz="-${x1} ${y1} ${z1}"/>
     <inertia ixx="${ixx1}" ixy="${ixy1}" ixz="${ixz1}" iyy="${iyy1}" iyz="${iyz1}" izz="${izz1}"/>
   </xacro:first_leg>
@@ -42,5 +47,6 @@
     <origin xyz="${joint_x1} ${joint_y1} ${joint_z1}" rpy="0 0 0"/>
     <origin xyz="-${visual_x1} -${visual_y1} -${visual_z1}"/>
-    <origin xyz="${x1} ${y1} ${z1}"/>
+    <origin xyz="-${visual_x1} -${visual_y1} -${visual_z1}"/>
+    <origin xyz="-${x1} -${y1} ${z1}"/>
     <inertia ixx="${ixx1}" ixy="${ixy1}" ixz="${ixz1}" iyy="${iyy1}" iyz="${iyz1}" izz="${izz1}"/>
   </xacro:first_leg>
@@ -48,5 +54,6 @@
     <origin xyz="-${joint_x1} -${joint_y1} ${joint_z1}" rpy="0 0 0"/>
     <origin xyz="${visual_x1} ${visual_y1} -${visual_z1}"/>
-    <origin xyz="-${x1} -${y1} ${z1}"/>
+    <origin xyz="${visual_x1} ${visual_y1} -${visual_z1}"/>
+    <origin xyz="${x1} ${y1} ${z1}"/>
     <inertia ixx="${ixx1}" ixy="-${ixy1}" ixz="${ixz1}" iyy="${iyy1}" iyz="${iyz1}" izz="${izz1}"/>
   </xacro:first_leg>
@@ -54,5 +61,6 @@
     <origin xyz="-${joint_x1} ${joint_y1} ${joint_z1}" rpy="0 0 0"/>
     <origin xyz="${visual_x1} -${visual_y1} -${visual_z1}"/>
-    <origin xyz="-${x1} ${y1} ${z1}"/>
+    <origin xyz="${visual_x1} -${visual_y1} -${visual_z1}"/>
+    <origin xyz="${x1} -${y1} ${z1}"/>
     <inertia ixx="${ixx1}" ixy="-${ixy1}" ixz="${ixz1}" iyy="${iyy1}" iyz="${iyz1}" izz="${izz1}"/>
   </xacro:first_leg>
@@ -60,5 +68,6 @@
     <origin xyz="${joint_x2} -${joint_y2} ${joint_z2}" rpy="0 0 0"/>
     <origin xyz="-${visual_x2} ${visual_y2} ${visual_z2}"/>
-    <origin xyz="${x2} -${y2} ${z2}"/>
+    <origin xyz="-${visual_x2} ${visual_y2} ${visual_z2}"/>
+    <origin xyz="${x2} ${y2} ${z2}"/>
     <inertia ixx="${ixx2}" ixy="${ixy2}" ixz="-${ixz2}" iyy="${iyy2}" iyz="${iyz2}" izz="${izz2}"/>
   </xacro:second_leg>
@@ -66,5 +75,6 @@
     <origin xyz="${joint_x2} ${joint_y2} ${joint_z2}" rpy="0 0 0"/>
     <origin xyz="-${visual_x2} -${visual_y2} ${visual_z2}"/>
-    <origin xyz="${x2} ${y2} ${z2}"/>
+    <origin xyz="-${visual_x2} -${visual_y2} ${visual_z2}"/>
+    <origin xyz="-${x2} -${y2} ${z2}"/>
     <inertia ixx="${ixx2}" ixy="${ixy2}" ixz="${ixz2}" iyy="${iyy2}" iyz="-${iyz2}" izz="${izz2}"/>
   </xacro:second_leg>
@@ -72,5 +82,6 @@
     <origin xyz="-${joint_x2} -${joint_y2} ${joint_z2}" rpy="0 0 0"/>
     <origin xyz="${visual_x2} ${visual_y2} ${visual_z2}"/>
-    <origin xyz="-${x2} -${y2} ${z2}"/>
+    <origin xyz="${visual_x2} ${visual_y2} ${visual_z2}"/>
+    <origin xyz="${x2} ${y2} ${z2}"/>
     <inertia ixx="${ixx2}" ixy="${ixy2}" ixz="-${ixz2}" iyy="${iyy2}" iyz="${iyz2}" izz="${izz2}"/>
   </xacro:second_leg>
@@ -78,5 +89,6 @@
     <origin xyz="-${joint_x2} ${joint_y2} ${joint_z2}" rpy="0 0 0"/>
     <origin xyz="${visual_x2} -${visual_y2} ${visual_z2}"/>
-    <origin xyz="-${x2} ${y2} ${z2}"/>
+    <origin xyz="${visual_x2} -${visual_y2} ${visual_z2}"/>
+    <origin xyz="${x2} -${y2} ${z2}"/>
     <inertia ixx="${ixx2}" ixy="${ixy2}" ixz="${ixz2}" iyy="${iyy2}" iyz="-${iyz2}" izz="${izz2}"/>
   </xacro:second_leg>
@@ -84,5 +96,6 @@
     <origin xyz="${joint_x3} -${joint_y3} ${joint_z3}" rpy="0 0 0"/>
     <origin xyz="-${visual_x3} ${visual_y3} ${visual_z3}"/>
-    <origin xyz="${x3} -${y3} ${z3}"/>
+    <origin xyz="-${visual_x3} ${visual_y3} ${visual_z3}"/>
+    <origin xyz="${x3} ${y3} ${z3}"/>
     <inertia ixx="${ixx3}" ixy="${ixy3}" ixz="-${ixz3}" iyy="${iyy3}" iyz="${iyz3}" izz="${izz3}"/>
   </xacro:third_leg>
@@ -90,5 +103,6 @@
     <origin xyz="${joint_x3} ${joint_y3} ${joint_z3}" rpy="0 0 0"/>
     <origin xyz="-${visual_x3} -${visual_y3} ${visual_z3}"/>
-    <origin xyz="${x3} ${y3} ${z3}"/>
+    <origin xyz="-${visual_x3} -${visual_y3} ${visual_z3}"/>
+    <origin xyz="${x3} -${y3} ${z3}"/>
     <inertia ixx="${ixx3}" ixy="${ixy3}" ixz="${ixz3}" iyy="${iyy3}" iyz="-${iyz3}" izz="${izz3}"/>
   </xacro:third_leg>
@@ -96,5 +110,6 @@
     <origin xyz="-${joint_x3} -${joint_y3} ${joint_z3}" rpy="0 0 0"/>
     <origin xyz="${visual_x3} ${visual_y3} ${visual_z3}"/>
-    <origin xyz="-${x3} -${y3} ${z3}"/>
+    <origin xyz="${visual_x3} ${visual_y3} ${visual_z3}"/>
+    <origin xyz="${x3} ${y3} ${z3}"/>
     <inertia ixx="${ixx3}" ixy="${ixy3}" ixz="-${ixz3}" iyy="${iyy3}" iyz="${iyz3}" izz="${izz3}"/>
   </xacro:third_leg>
@@ -102,5 +117,6 @@
     <origin xyz="-${joint_x3} ${joint_y3} ${joint_z3}" rpy="0 0 0"/>
     <origin xyz="${visual_x3} -${visual_y3} ${visual_z3}"/>
-    <origin xyz="-${x3} ${y3} ${z3}"/>
+    <origin xyz="${visual_x3} -${visual_y3} ${visual_z3}"/>
+    <origin xyz="${x3} -${y3} ${z3}"/>
     <inertia ixx="${ixx3}" ixy="${ixy3}" ixz="${ixz3}" iyy="${iyy3}" iyz="-${iyz3}" izz="${izz3}"/>
   </xacro:third_leg>
@@ -131,9 +147,4 @@
   <xacro:leg_trans prefix="D3"/>
   <!-- =============== Gazebo =============== -->
-  <gazebo>
-    <plugin name="gazebo_ros_control" filename="libgazebo_ros_control.so">
-      <!-- <robotNamespace>fourth_robot</robotNamespace> -->
-    </plugin>
-  </gazebo>
   <!-- Body -->
   <gazebo>

File: dream_walker_description/urdf/leg/leg.param.xacro (robot description, xacro)
@@ -5,19 +5,19 @@
   <property name="mass2" value="3.66"/>
   <property name="mass3" value="1.72"/>
-  <property name="x0" value="0.26100"/>
-  <property name="x1" value="0.11810"/>
-  <property name="x2" value="0.00440"/>
-  <property name="x3" value="0.00000"/>
-  <property name="x4" value="0.00000"/>
-  <property name="y0" value="0.082980"/>
-  <property name="y1" value="0.001110"/>
-  <property name="y2" value="0.161810"/>
-  <property name="y3" value="0.111690"/>
-  <property name="y4" value="0.002140"/>
+  <property name="x0" value="0.03900"/>
+  <property name="x1" value="0.00440"/>
+  <property name="x2" value="0.0000"/>
+  <property name="x3" value="0.0000"/>
+  <property name="x4" value="0.0000"/>
+  <property name="y0" value="0.00002"/>
+  <property name="y1" value="0.00113"/>
+  <property name="y2" value="0.04882"/>
+  <property name="y3" value="0.00214"/>
+  <property name="y4" value="0.00000"/>
   <property name="z0" value="-0.00001"/>
-  <property name="z1" value="-0.00004"/>
-  <property name="z2" value="-0.09715"/>
-  <property name="z3" value="-0.41291"/>
-  <property name="z4" value="-0.25289"/>
+  <property name="z1" value="-0.00005"/>
+  <property name="z2" value="-0.09719"/>
+  <property name="z3" value="-0.19011"/>
+  <property name="z4" value="-0.00000"/>
   <property name="joint_x0" value="0.30000"/>
   <property name="joint_x1" value="0.08350"/>
@@ -71,3 +71,27 @@
   <property name="izz2" value="0.011896"/>
   <property name="izz3" value="0.001426"/>
+  <property name="ixx0a" value="0.01422"/>
+  <property name="ixx1a" value="0.00229"/>
+  <property name="ixx2a" value="0.075241"/>
+  <property name="ixx3a" value="0.026984"/>
+  <property name="ixy0a" value="0.038006"/>
+  <property name="ixy1a" value="0.000008"/>
+  <property name="ixy2a" value="0"/>
+  <property name="ixy3a" value="0"/>
+  <property name="ixz0a" value="0"/>
+  <property name="ixz1a" value="1.0E-06"/>
+  <property name="ixz2a" value="5.0E-06"/>
+  <property name="ixz3a" value="0"/>
+  <property name="iyy0a" value="0121986"/>
+  <property name="iyy1a" value="0.002657"/>
+  <property name="iyy2a" value="0.069683"/>
+  <property name="iyy3a" value="0.026649"/>
+  <property name="iyz0a" value="0.000002"/>
+  <property name="iyz1a" value="1.0E-06"/>
+  <property name="iyz2a" value="0.013776"/>
+  <property name="iyz3a" value="0.000717"/>
+  <property name="izz0a" value="0.134071"/>
+  <property name="izz1a" value="0.002511"/>
+  <property name="izz2a" value="0.011896"/>
+  <property name="izz3a" value="0.001426"/>
 </robot>

File: dream_walker_description/urdf/leg/leg.urdf.xacro (robot description, xacro)
@@ -5,5 +5,5 @@
   <xacro:include filename="$(find dream_walker_description)/urdf/leg/leg.transmission.xacro"/>
   <xacro:include filename="$(find dream_walker_description)/urdf/leg/color.xacro"/>
-  <xacro:macro name="zero_leg" params="prefix parent *joint_origin *visual_origin *inertial_origin *inertia">
+  <xacro:macro name="zero_leg" params="prefix parent *joint_origin *visual_origin *collision_origin  *inertial_origin *inertia">
     <joint name="${prefix}_joint" type="fixed">
       <insert_block name="joint_origin"/>
@@ -21,4 +21,5 @@
       </visual>
       <collision>
+        <insert_block name="collision_origin"/>
         <geometry>
           <mesh filename="package://dream_walker_description/meshes/${prefix}_link.STL"/>
@@ -32,5 +33,5 @@
     </link>
   </xacro:macro>
-  <xacro:macro name="first_leg" params="prefix parent *joint_origin *visual_origin *inertial_origin *inertia">
+  <xacro:macro name="first_leg" params="prefix parent *joint_origin *visual_origin *collision_origin *inertial_origin *inertia">
     <joint name="${prefix}_joint" type="revolute">
       <insert_block name="joint_origin"/>
@@ -49,4 +50,5 @@
       </visual>
       <collision>
+        <insert_block name="collision_origin"/>
         <geometry>
           <mesh filename="package://dream_walker_description/meshes/${prefix}_link.STL"/>
@@ -60,5 +62,5 @@
     </link>
   </xacro:macro>
-  <xacro:macro name="second_leg" params="prefix parent *joint_origin *visual_origin *inertial_origin *inertia">
+  <xacro:macro name="second_leg" params="prefix parent *joint_origin *visual_origin *collision_origin *inertial_origin *inertia">
     <joint name="${prefix}_joint" type="revolute">
       <insert_block name="joint_origin"/>
@@ -77,4 +79,5 @@
       </visual>
       <collision>
+        <insert_block name="collision_origin"/>
         <geometry>
           <mesh filename="package://dream_walker_description/meshes/${prefix}_link.STL"/>
@@ -88,5 +91,5 @@
     </link>
   </xacro:macro>
-  <xacro:macro name="third_leg" params="prefix parent *joint_origin *visual_origin *inertial_origin *inertia">
+  <xacro:macro name="third_leg" params="prefix parent *joint_origin *visual_origin *collision_origin *inertial_origin *inertia">
     <joint name="${prefix}_joint" type="revolute">
       <insert_block name="joint_origin"/>
@@ -105,4 +108,5 @@
       </visual>
       <collision>
+        <insert_block name="collision_origin"/>
         <geometry>
           <mesh filename="package://dream_walker_description/meshes/${prefix}_link.STL"/>
